Commit message: tool_urdf_added but gzserver error

File: iiwa_description/urdf/iiwa14.xacro (robot description, xacro)
@@ -120,5 +120,5 @@
           <mesh filename="package://iiwa_description/meshes/iiwa14/visual/link_1.stl"/>
         </geometry>
-        <material name="Orange"/>
+        <material name="White"/>
       </visual>
       <collision>
@@ -127,5 +127,5 @@
           <mesh filename="package://iiwa_description/meshes/iiwa14/collision/link_1${collision_postfix}.stl"/>
         </geometry>
-        <material name="Orange"/>
+        <material name="White"/>
       </collision>
     </link>
@@ -156,5 +156,5 @@
           <mesh filename="package://iiwa_description/meshes/iiwa14/visual/link_2.stl"/>
         </geometry>
-        <material name="Orange"/>
+        <material name="White"/>
       </visual>
       <collision>
@@ -163,5 +163,5 @@
           <mesh filename="package://iiwa_description/meshes/iiwa14/collision/link_2${collision_postfix}.stl"/>
         </geometry>
-        <material name="Orange"/>
+        <material name="White"/>
       </collision>
     </link>
@@ -192,5 +192,5 @@
           <mesh filename="package://iiwa_description/meshes/iiwa14/visual/link_3.stl"/>
         </geometry>
-        <material name="Orange"/>
+        <material name="White"/>
       </visual>
       <collision>
@@ -199,5 +199,5 @@
           <mesh filename="package://iiwa_description/meshes/iiwa14/collision/link_3${collision_postfix}.stl"/>
         </geometry>
-        <material name="Orange"/>
+        <material name="White"/>
       </collision>
     </link>
@@ -228,5 +228,5 @@
           <mesh filename="package://iiwa_description/meshes/iiwa14/visual/link_4.stl"/>
         </geometry>
-        <material name="Orange"/>
+        <material name="White"/>
       </visual>
       <collision>
@@ -235,5 +235,5 @@
           <mesh filename="package://iiwa_description/meshes/iiwa14/collision/link_4${collision_postfix}.stl"/>
         </geometry>
-        <material name="Orange"/>
+        <material name="White"/>
       </collision>
     </link>
@@ -264,5 +264,5 @@
           <mesh filename="package://iiwa_description/meshes/iiwa14/visual/link_5.stl"/>
         </geometry>
-        <material name="Orange"/>
+        <material name="White"/>
       </visual>
       <collision>
@@ -271,5 +271,5 @@
           <mesh filename="package://iiwa_description/meshes/iiwa14/collision/link_5${collision_postfix}.stl"/>
         </geometry>
-        <material name="Orange"/>
+        <material name="White"/>
       </collision>
     </link>
@@ -300,5 +300,5 @@
           <mesh filename="package://iiwa_description/meshes/iiwa14/visual/link_6.stl"/>
         </geometry>
-        <material name="Orange"/>
+        <material name="White"/>
       </visual>
       <collision>
@@ -307,5 +307,5 @@
           <mesh filename="package://iiwa_description/meshes/iiwa14/collision/link_6${collision_postfix}.stl"/>
         </geometry>
-        <material name="Orange"/>
+        <material name="White"/>
       </collision>
     </link>
