Commit message: simulation working

File: iiwa_description/urdf/iiwa14_rs_tool.urdf.xacro (robot description, xacro)
@@ -5,8 +5,5 @@
   <xacro:include filename="$(find iiwa_description)/urdf/materials.xacro" />
   <!--Import the iiwa14 macro -->
-  <xacro:include filename="$(find iiwa_description)/urdf/iiwa14.xacro"/>
-  <!--Import the rs_tool macro -->
-  <xacro:include filename="$(find iiwa_description)/urdf/rs_tool.xacro"/>
-  <!-- <xacro:include filename="$(find iiwa_description)/urdf/rs_camera_ee.urdf.xacro"/> -->
+  <xacro:include filename="$(find iiwa_description)/urdf/iiwa14_rs_tool.xacro"/>
   <!--  Arguments for the iiwa14 macro  -->
   <xacro:arg name="hardware_interface" default="PositionJointInterface"/>

File: iiwa_description/urdf/objects/human.urdf (robot description, URDF)
Before this commit: robot human_in_gazebo, 2 links, 1 joints
Joints:
- joint human_on_world: origin xyz=0.05 -0.75 0.0 rpy=0 0 0 -> xyz=0.5 -0.5 0.05 rpy=0 0 0

File: iiwa_description/urdf/realsense/_d435.urdf.xacro (robot description, xacro)
@@ -10,5 +10,5 @@
   <!-- <xacro:include filename="$(find realsense2_description)/urdf/_materials.urdf.xacro" />
   <xacro:include filename="$(find realsense2_description)/urdf/_usb_plug.urdf.xacro" /> -->
-  <xacro:include filename="$(find iiwa_description)/urdf/_d435.gazebo.xacro"/>
+  <xacro:include filename="$(find iiwa_description)/urdf/realsense/_d435.gazebo.xacro"/>
   <xacro:macro name="sensor_d435" params="parent *origin name:=camera topics_ns:=camera
    use_nominal_extrinsics:=false add_plug:=false use_mesh:=true">

File: iiwa_description/urdf/realsense/rs_camera_ee.urdf.xacro (robot description, xacro)
@@ -2,5 +2,5 @@
 <robot name="realsense2_camera" xmlns:xacro="http://www.ros.org/wiki/xacro">
   <xacro:arg name="use_nominal_extrinsics" default="false" />
-  <xacro:include filename="$(find iiwa_description)/urdf/_d435.urdf.xacro"/>
+  <xacro:include filename="$(find iiwa_description)/urdf/realsense/_d435.urdf.xacro"/>
   <!-- <xacro:include filename="$(find iiwa_description)/urdf/_d435i.urdf.xacro"/> -->
   <xacro:sensor_d435 parent="tool_link" use_nominal_extrinsics="$(arg use_nominal_extrinsics)" name="camera">

File: iiwa_description/urdf/realsense/rs_tool.xacro (robot description, xacro)
@@ -2,5 +2,5 @@
 <robot name="rs_tool" xmlns:xacro="http://www.ros.org/wiki/xacro">
 <!-- Tool properties -->
-  <!-- <xacro:property name="tool_mass" value="0.050" /> -->
+  <xacro:property name="tool_mass" value="0.050" />
   <!--property name="tool_joint_offset" value="0.00 0.00 0.00" /-->
   <!--property name="tool_link_offset" value="0.00 0.00 0.10" /-->
@@ -18,6 +18,6 @@
       <origin xyz="0 0 0" rpy="0 0 0"/>
       <geometry>
-	      <!-- <mesh filename="package://iiwa_description/meshes/tools/visual/rscamera_tool.STL"/> -->
-		<cylinder length="0.1275" radius="0.020"/>
+	      <mesh filename="package://iiwa_description/meshes/tools/visual/rscamera_tool.STL"/>
+		<!-- <cylinder length="0.1275" radius="0.020"/> -->
       </geometry>
       <material name="Grey"/>
@@ -26,6 +26,6 @@
       <origin xyz="0 0 0" rpy="0 0 0"/>
       <geometry>
-        <!-- <mesh filename="package://iiwa_description/meshes/tools/collision/rscamera_tool.STL"/> -->
-		<cylinder length="0.1275" radius="0.020"/>
+        <mesh filename="package://iiwa_description/meshes/tools/collision/rscamera_tool.STL"/>
+		<!-- <cylinder length="0.1275" radius="0.020"/> -->
       </geometry>
       <material name="Grey"/>
