Commit message: adding urdf_tera_tool

File: iiwa_description/urdf/iiwa14_rs_tool.xacro (robot description, xacro)
@@ -358,5 +358,6 @@
       </inertial>
     </link>
-    <xacro:include filename="$(find iiwa_description)/urdf/realsense/rs_tool.xacro"/>
+    <!-- <xacro:include filename="$(find iiwa_description)/urdf/realsense/rs_tool.xacro"/>  -->
+    <xacro:include filename="$(find iiwa_description)/urdf/realsense/rs_tera_tool.xacro"/>
     <xacro:include filename="$(find iiwa_description)/urdf/realsense/rs_camera_ee.urdf.xacro"/>
     <!--Extensions -->

File: iiwa_description/urdf/realsense/rs_tera_tool.xacro (robot description, xacro)
@@ -16,8 +16,8 @@
   <link name="tool_link">
     <visual>
-      <origin xyz="0 0 0" rpy="0 0 0"/>
+      <origin xyz="-0.120 0.038 0" rpy="0 0 0"/>
       <geometry>
-	      <mesh filename="package://iiwa_description/meshes/tools/visual/rscamera_tool.STL"/>
-        <!-- <mesh filename="package://iiwa_description/meshes/tools/visual/rs_tera_tool_urdf.STL"/> -->
+	      <!-- <mesh filename="package://iiwa_description/meshes/tools/visual/rscamera_tool.STL"/> -->
+        <mesh filename="package://iiwa_description/meshes/tools/visual/rs_tera_tool_urdf.STL"/>
 		<!-- <cylinder length="0.1275" radius="0.020"/> -->
       </geometry>
@@ -25,8 +25,8 @@
     </visual>
     <collision>
-      <origin xyz="0 0 0" rpy="0 0 0"/>
+      <origin xyz="-0.120 0.038 0" rpy="0 0 0"/>
       <geometry>
-        <mesh filename="package://iiwa_description/meshes/tools/collision/rscamera_tool.STL"/>
-        <!-- <mesh filename="package://iiwa_description/meshes/tools/visual/rs_tera_tool_urdf.STL"/> -->
+        <!-- <mesh filename="package://iiwa_description/meshes/tools/collision/rscamera_tool.STL"/> -->
+        <mesh filename="package://iiwa_description/meshes/tools/visual/rs_tera_tool_urdf.STL"/>
 		<!-- <cylinder length="0.1275" radius="0.020"/> -->
       </geometry>
@@ -38,5 +38,5 @@
     <parent link="tool_link" />
     <child link = "tool_link_ee" />
-    <origin xyz="0.03 0.08 0.1" rpy="0 0 0" />
+    <origin xyz="0.03 0.08 0.225" rpy="0 0 0" />
   </joint>
   <!--  The TCP frame is here defined -->
